File: PCB/MK I/TB315A56612FNG_TO_THT/TB315A56612FNG_TO_THT.kicad_sch (KiCad schematic)
At the start: 16 parts, among them J1 Conn_01x06_Pin, J2 Conn_01x06_Pin, J3 Conn_01x06_Pin, J4 Conn_01x06_Pin, J5 Conn_01x02_Pin, J8 Conn_01x15_Pin, J9 Conn_01x15_Pin, U1 TB6612FNG, U2 LM1086, U3 TSOP382xx

Commit message: ki cad
savva mi bnarval do prdele curaka
Parts:
- removed J8, J9: Conn_01x15_Pin, symbol Connector:Conn_01x15_Pin
- added U4: DEVKIT_V1_ESP32-WROOM-32, lf_zetor_board:MODULE_DEVKIT_V1_ESP32-WROOM-32, symbol lf_zetor_kicad_sch:DEVKIT_V1_ESP32-WROOM-32
Other:
- note added: "vstup ze senzoru"

Commit message: pluh
mk update
Parts:
- added J6, J8: Conn_01x06_Pin, Connector_JST:JST_XH_B6B-XH-A_1x06_P2.50mm_Vertical, symbol Connector:Conn_01x06_Pin
- added R1, R11, R13, R15, R17, R3, R5, R7, R9: 100R, Resistor_SMD:R_0805_2012Metric, symbol Device:R
- added R10, R12, R14, R16, R18, R2, R4, R6, R8: 10k, Resistor_SMD:R_0805_2012Metric, symbol Device:R
- added U10, U11, U12, U13, U5, U6, U7, U8, U9: QRE1113GR, OptoDevice:OnSemi_CASE100CY, symbol Sensor_Proximity:QRE1113GR
Connections:
- net GND: now also U10.2 (K), U10.4, U11.2 (K), U11.4, U12.2 (K), U12.4, U13.2 (K), U13.4, U5.2 (K), U5.4, U6.2 (K), U6.4, U7.2 (K), U7.4, U8.2 (K), U8.4, U9.2 (K), U9.4
- new net: R9.2, U12.1 (A)
- new net: R15.2, U10.1 (A)
- new net: R1.2, U7.1 (A)
- new net: R11.2, U9.1 (A)
- new net: R13.2, U13.1 (A)
- new net: R3.2, U5.1 (A)
- new net: R7.2, U6.1 (A)
- new net: R5.2, U8.1 (A)
- new net: R17.2, U11.1 (A)
- new net Sen1Out: R2.1, U7.3
- new net Sen2Out: R4.1, U5.3
- new net Sen3Out: R6.1, U8.3
- new net Sen4Out: R8.1, U6.3
- new net Sen5Out: R10.1, U12.3
- new net Sen6Out: R12.1, U9.3
- new net Sen7Out: R14.1, U13.3
- new net Sen8Out: R16.1, U10.3
- new net Sen9Out: R18.1, U11.3
- new net VCC: R1.1, R10.2, R11.1, R12.2, R13.1, R14.2, R15.1, R16.2, R17.1, R18.2, R2.2, R3.1, R4.2, R5.1, R6.2, R7.1, R8.2, R9.1
Other:
- note added: "16 pouzitelnych pinu"
- note added: "driver na motory 2 pwm 2 smer A 2 smer B"
- note added: "ir senzor 1 vypinac elektricky"
- note added: "motor output/input with encoder encouder"
- note added: "senzor pin 9"
- note removed: "motor output through encouder"

Commit message: ehhh
eeeeh
Parts:
- removed C1, C3: 100nF, symbol Device:C
- removed C2, C4, C6, C8: 10uF, symbol Device:C_Polarized
- removed J1, J4: Conn_01x06_Pin, symbol Connector:Conn_01x06_Pin
- removed J2, J3: Conn_01x06_Pin, Connector_JST:JST_SH_BM06B-SRSS-TB_1x06-1MP_P1.00mm_Vertical, symbol Connector:Conn_01x06_Pin
- removed J5: Conn_01x02_Pin, symbol Connector:Conn_01x02_Pin
- removed J6, J8: Conn_01x06_Pin, Connector_JST:JST_XH_B6B-XH-A_1x06_P2.50mm_Vertical, symbol Connector:Conn_01x06_Pin
- removed R1, R11, R13, R15, R17, R3, R5, R7, R9: 100R, Resistor_SMD:R_0805_2012Metric, symbol Device:R
- removed R10, R12, R14, R16, R18, R2, R4, R6, R8: 10k, Resistor_SMD:R_0805_2012Metric, symbol Device:R
- removed U1: TB6612FNG, Package_SO:SSOP-24_5.3x8.2mm_P0.65mm, symbol Driver_Motor:TB6612FNG
- removed U10, U11, U12, U13, U5, U6, U7, U8, U9: QRE1113GR, OptoDevice:OnSemi_CASE100CY, symbol Sensor_Proximity:QRE1113GR
- removed U2: LM1086, Package_TO_SOT_THT:TO-220-3_Vertical, symbol Regulator_Linear:LM317_TO-220
- removed U3: TSOP382xx, OptoDevice:Vishay_MINICAST-3Pin, symbol Interface_Optical:TSOP382xx
- removed U4: DEVKIT_V1_ESP32-WROOM-32, lf_zetor_board:MODULE_DEVKIT_V1_ESP32-WROOM-32, symbol lf_zetor_kicad_sch:DEVKIT_V1_ESP32-WROOM-32
Other:
- added sheet main board (untitled.kicad_sch)
- added sheet senzor ring (../senzor_ring/senzor_ring.kicad_sch)
- note removed: "16 pouzitelnych pinu"
- note removed: "driver - for - motors"
- note removed: "driver na motory 2 pwm 2 smer A 2 smer B"
- note removed: "esp - pin out dodelat"
- note removed: "ir senzor 1 vypinac elektricky"
- note removed: "li-po akumulator"
- note removed: "motor output/input with encoder encouder"
- note removed: "power - suply"
- note removed: "regulator 12 - 5 V"
- note removed: "senzor pin 9"
- note removed: "tsop setup"
- note removed: "vstup ze senzoru"
