File: PCB/MK I/TB315A56612FNG_TO_THT/_autosave-TB315A56612FNG_TO_THT.kicad_pcb (KiCad board)
At the start: 2 copper layers, 120 x 65 mm, 36 parts, among them J1 Conn_01x06_Pin, J10 Conn_01x06_Pin, J2 Conn_01x06_Pin, J3 Conn_01x06_Pin, J4 Conn_01x06_Pin, J9 Conn_01x06_Pin, U1 QRE1113GR, U10 QRE1113GR, U11 QRE1113GR, U12 QRE1113GR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

Commit message: saveee
s
Parts:
- added J5: Conn_01x19_Pin, Connector_PinHeader_2.54mm:PinHeader_1x19_P2.54mm_Vertical, F.Cu at (85.1, 80.4)
- added J6: Conn_01x19_Pin, Connector_PinHeader_2.54mm:PinHeader_1x19_P2.54mm_Vertical, F.Cu at (89.7, 80.4)
- J2, J4: footprint Connector_JST:JST_SH_BM06B-SRSS-TB_1x06-1MP_P1.00mm_Vertical -> Connector_JST:JST_XH_B6B-XH-A_1x06_P2.50mm_Vertical
Connections:
- J1 pad 1: unconnected-(J1-Pin_1-Pad1) -> Sen5Out
- J1 pad 2: unconnected-(J1-Pin_2-Pad2) -> Sen4Out
- J1 pad 3: unconnected-(J1-Pin_3-Pad3) -> Sen3Out
- J1 pad 4: unconnected-(J1-Pin_4-Pad4) -> Sen2Out
- J1 pad 5: unconnected-(J1-Pin_5-Pad5) -> Sen1Out
- J1 pad 6: unconnected-(J1-Pin_6-Pad6) -> GND
- J10 pad 1: unconnected-(J10-Pin_1-Pad1) -> +5V
- J10 pad 2: unconnected-(J10-Pin_2-Pad2) -> S_D9
- J10 pad 3: unconnected-(J10-Pin_3-Pad3) -> S_D8
- J10 pad 4: unconnected-(J10-Pin_4-Pad4) -> S_D7
- J10 pad 5: unconnected-(J10-Pin_5-Pad5) -> S_D6
- J10 pad 6: unconnected-(J10-Pin_6-Pad6) -> GND
- J2 pad 1: unconnected-(J2-Pin_1-Pad1) -> LM1
- J2 pad 2: unconnected-(J2-Pin_2-Pad2) -> LM2
- J3 pad 1: unconnected-(J3-Pin_1-Pad1) -> VCC
- J3 pad 2: unconnected-(J3-Pin_2-Pad2) -> Sen6Out
- J3 pad 3: unconnected-(J3-Pin_3-Pad3) -> Sen7Out
- J3 pad 4: unconnected-(J3-Pin_4-Pad4) -> Sen8Out
- J3 pad 5: unconnected-(J3-Pin_5-Pad5) -> Sen9Out
- J3 pad 6: unconnected-(J3-Pin_6-Pad6) -> GND
- J4 pad 5: unconnected-(J4-Pin_5-Pad5) -> RM1
- J4 pad 6: unconnected-(J4-Pin_6-Pad6) -> RM2
- J9 pad 1: unconnected-(J9-Pin_1-Pad1) -> S_D5
- J9 pad 2: unconnected-(J9-Pin_2-Pad2) -> S_D4
- J9 pad 3: unconnected-(J9-Pin_3-Pad3) -> S_D3
- J9 pad 4: unconnected-(J9-Pin_4-Pad4) -> S_D2
- J9 pad 5: unconnected-(J9-Pin_5-Pad5) -> S_D1
- J9 pad 6: unconnected-(J9-Pin_6-Pad6) -> GND
- U8 pad 1: Net-(U8-AO1-Pad1) -> LM1
- U8 pad 11: Net-(U8-BO1-Pad11) -> RM1
- U8 pad 12: Net-(U8-BO1-Pad11) -> RM1
- U8 pad 15: unconnected-(U8-PWMB-Pad15) -> PWM_B
- U8 pad 16: unconnected-(U8-BIN2-Pad16) -> D.M.C.B.2
- U8 pad 17: unconnected-(U8-BIN1-Pad17) -> D.M.C.B.1
- U8 pad 2: Net-(U8-AO1-Pad1) -> LM1
- U8 pad 21: unconnected-(U8-AIN1-Pad21) -> D.M.C.A.1
- U8 pad 22: unconnected-(U8-AIN2-Pad22) -> D.M.C.A.2
- U8 pad 23: unconnected-(U8-PWMA-Pad23) -> PWM_A
- U8 pad 3: Net-(U8-PGND1-Pad3) -> unconnected-(U8-PGND1-Pad3)_1
- U8 pad 4: Net-(U8-PGND1-Pad3) -> unconnected-(U8-PGND1-Pad3)
- U8 pad 5: Net-(U8-AO2-Pad5) -> LM2
- U8 pad 6: Net-(U8-AO2-Pad5) -> LM2
- U8 pad 7: Net-(U8-BO2-Pad7) -> RM2
- U8 pad 8: Net-(U8-BO2-Pad7) -> RM2
