File: PCB/MK I/TB315A56612FNG_TO_THT/TB315A56612FNG_TO_THT.kicad_pcb (KiCad board)
At the start: 2 copper layers, 0 parts

Commit message: ki cad
savva mi bnarval do prdele curaka
Parts:
- added J2: Conn_01x06_Pin, Connector_JST:JST_SH_BM06B-SRSS-TB_1x06-1MP_P1.00mm_Vertical, F.Cu at (45.2, 30.4)
- added J3: Conn_01x06_Pin, Connector_JST:JST_SH_BM06B-SRSS-TB_1x06-1MP_P1.00mm_Vertical, F.Cu at (45.2, 36.7)
- added U1: TB6612FNG, Package_SO:SSOP-24_5.3x8.2mm_P0.65mm, F.Cu at (45.1, 50.8)
- added U2: LM1086, Package_TO_SOT_THT:TO-220-3_Vertical, F.Cu at (43.0, 43.7)
- added U3: TSOP382xx, OptoDevice:Vishay_MINICAST-3Pin, F.Cu at (41.5, 58.0)
- added U4: DEVKIT_V1_ESP32-WROOM-32, lf_zetor_board:MODULE_DEVKIT_V1_ESP32-WROOM-32, F.Cu at (202.3, 78.8)
Other:
- board outline added: 120 x 65 mm

Commit message: Patch some shits
Potřeby jemně předělat senzor
Parts:
- added C10: 10uF, Capacitor_SMD:CP_Elec_4x5.4, F.Cu at (58.0, 79.5)
- added C11: 100nF, Capacitor_Tantalum_SMD:CP_EIA-7343-31_Kemet-D, F.Cu at (91.5, 85.5)
- added C12: 10uF, Capacitor_SMD:CP_Elec_4x5.4, F.Cu at (91.5, 79.0)
- added C5: 100nF, Capacitor_Tantalum_SMD:CP_EIA-7343-31_Kemet-D, F.Cu at (110.8, 83.6)
- added C7: 10uF, Capacitor_SMD:CP_Elec_4x5.4, F.Cu at (116.5, 84.0)
- added C9: 10uF, Capacitor_SMD:CP_Elec_4x5.4, F.Cu at (67.6, 36.8)
- added J1: Conn_01x06_Pin, Connector_JST:JST_GH_SM06B-GHS-TB_1x06-1MP_P1.25mm_Horizontal, F.Cu at (208.5, 40.2)
- added J10: Conn_01x06_Pin, Connector_JST:JST_XH_B6B-XH-A_1x06_P2.50mm_Vertical, F.Cu at (52.9, 54.9)
- added J4: Conn_01x06_Pin, Connector_JST:JST_GH_SM06B-GHS-TB_1x06-1MP_P1.25mm_Horizontal, F.Cu at (241.8, 130.0)
- added J5: Conn_01x19_Pin, Connector_PinHeader_2.54mm:PinHeader_1x19_P2.54mm_Vertical, F.Cu at (195.3, 88.5)
- added J6: Conn_01x19_Pin, Connector_PinHeader_2.54mm:PinHeader_1x19_P2.54mm_Vertical, F.Cu at (220.5, 88.6)
- added J7: Conn_01x02_Pin, Connector_AMASS:AMASS_XT30PW-M_1x02_P2.50mm_Horizontal, F.Cu at (89.0, 91.1)
- added J9: Conn_01x06_Pin, Connector_JST:JST_XH_B6B-XH-A_1x06_P2.50mm_Vertical, F.Cu at (47.8, 47.0)
- added R1: 100R, Resistor_SMD:R_0805_2012Metric, F.Cu at (137.7, 37.9)
- added R10: 100R, Resistor_SMD:R_0805_2012Metric, F.Cu at (124.7, 29.6)
- added R11: 100R, Resistor_SMD:R_0805_2012Metric, F.Cu at (124.7, 32.5)
- added R12: 100R, Resistor_SMD:R_0805_2012Metric, F.Cu at (124.7, 35.5)
- added R13: 100R, Resistor_SMD:R_0805_2012Metric, F.Cu at (124.7, 38.4)
- added R14: 10k, Resistor_SMD:R_0805_2012Metric, F.Cu at (124.7, 41.4)
- added R15: 10k, Resistor_SMD:R_0805_2012Metric, F.Cu at (129.2, 23.6)
- added R16: 10k, Resistor_SMD:R_0805_2012Metric, F.Cu at (129.2, 26.6)
- added R17: 10k, Resistor_SMD:R_0805_2012Metric, F.Cu at (129.2, 29.6)
- added R18: 10k, Resistor_SMD:R_0805_2012Metric, F.Cu at (129.2, 32.5)
- added R2: 100R, Resistor_SMD:R_0805_2012Metric, F.Cu at (120.3, 26.6)
- added R3: 100R, Resistor_SMD:R_0805_2012Metric, F.Cu at (120.3, 29.6)
- added R4: 100R, Resistor_SMD:R_0805_2012Metric, F.Cu at (120.3, 32.5)
- added R5: 10k, Resistor_SMD:R_0805_2012Metric, F.Cu at (120.3, 35.5)
- added R6: 10k, Resistor_SMD:R_0805_2012Metric, F.Cu at (120.3, 38.4)
- added R7: 10k, Resistor_SMD:R_0805_2012Metric, F.Cu at (120.3, 41.4)
- added R8: 10k, Resistor_SMD:R_0805_2012Metric, F.Cu at (124.7, 23.6)
- added R9: 100R, Resistor_SMD:R_0805_2012Metric, F.Cu at (124.7, 26.6)
- added SW1: SW_DPDT, lf_zetor_board:255SB, F.Cu at (168.0, 145.5)
- added U10: LM1086, Package_TO_SOT_THT:TO-220-3_Vertical, F.Cu at (108.2, 93.7)
- added U11: TSOP382xx, OptoDevice:Vishay_MINICAST-3Pin, F.Cu at (203.7, 145.5)
- added U12: QRE1113GR, OptoDevice:OnSemi_CASE100CY, F.Cu at (256.4, 37.8)
- added U13: QRE1113GR, OptoDevice:OnSemi_CASE100CY, F.Cu at (230.4, 33.0)
- added U5: QRE1113GR, OptoDevice:OnSemi_CASE100CY, F.Cu at (217.4, 33.0)
- added U7: QRE1113GR, OptoDevice:OnSemi_CASE100CY, F.Cu at (243.4, 34.5)
- added U8: TB6612FNG, Package_SO:SSOP-24_5.3x8.2mm_P0.65mm, F.Cu at (206.2, 138.0)
- added U9: QRE1113GR, OptoDevice:OnSemi_CASE100CY, F.Cu at (269.4, 43.2)
- J2, J3: footprint Connector_JST:JST_SH_BM06B-SRSS-TB_1x06-1MP_P1.00mm_Vertical -> Connector_JST:JST_GH_SM06B-GHS-TB_1x06-1MP_P1.25mm_Horizontal
- U1: value TB6612FNG -> QRE1113GR; footprint Package_SO:SSOP-24_5.3x8.2mm_P0.65mm -> OptoDevice:OnSemi_CASE100CY
- U2: value LM1086 -> QRE1113GR; footprint Package_TO_SOT_THT:TO-220-3_Vertical -> OptoDevice:OnSemi_CASE100CY
- U3: value TSOP382xx -> QRE1113GR; footprint OptoDevice:Vishay_MINICAST-3Pin -> OptoDevice:OnSemi_CASE100CY
- U4: value DEVKIT_V1_ESP32-WROOM-32 -> QRE1113GR; footprint lf_zetor_board:MODULE_DEVKIT_V1_ESP32-WROOM-32 -> OptoDevice:OnSemi_CASE100CY
- moved J3 175.7 mm to (220.9, 40.3)
- moved J2 160.1 mm to (170.8, 129.8), turned to -90 degrees
- moved U3 151.8 mm to (191.4, 34.5)
- moved U2 135.6 mm to (178.4, 37.8)
- moved U1 120.6 mm to (165.4, 43.2)
- moved U4 45.8 mm to (204.4, 33.1)
Connections:
- J2 pad 1: Net-(J1-Pin_1) -> LM1
- J2 pad 2: Net-(J1-Pin_2) -> LM2
- J2 pad 3: Net-(J1-Pin_3) -> unconnected-(J2-Pin_3-Pad3)
- J2 pad 4: Net-(J1-Pin_4) -> unconnected-(J2-Pin_4-Pad4)
- J2 pad 5: Net-(J1-Pin_5) -> unconnected-(J2-Pin_5-Pad5)
- J2 pad 6: Net-(J1-Pin_6) -> unconnected-(J2-Pin_6-Pad6)
- J3 pad 1: Net-(J3-Pin_1) -> VCC
- J3 pad 2: Net-(J3-Pin_2) -> Sen9Out
- J3 pad 3: Net-(J3-Pin_3) -> Sen8Out
- J3 pad 4: Net-(J3-Pin_4) -> Sen7Out
- J3 pad 5: Net-(J3-Pin_5) -> Sen6Out
- J3 pad 6: Net-(J3-Pin_6) -> GND
- U1 pad 1: Net-(U1-AO1-Pad1) -> Net-(U1-A)
- U1 pad 2: Net-(U1-AO1-Pad1) -> GND
- U1 pad 3: Net-(U1-PGND1-Pad3) -> Sen1Out
- U1 pad 4: Net-(U1-PGND1-Pad3) -> GND
- U2 pad 1: GND -> Net-(U2-A)
- U2 pad 2: +5V -> GND
- U2 pad 3: +12V -> Sen2Out
- U3 pad 1: D-pin-ESP -> Net-(U3-A)
- U3 pad 3: +5V -> Sen3Out
- U4 pad 1: unconnected-(U4-3V3-Pad1) -> Net-(U4-A)
- U4 pad 2: unconnected-(U4-EN-Pad2) -> GND
- U4 pad 3: unconnected-(U4-SENSOR_VP-Pad3) -> Sen4Out
- U4 pad 4: unconnected-(U4-SENSOR_VN-Pad4) -> GND
Other:
- board size 120 x 65 mm -> 128.7 x 121.5 mm

Commit message: pcb shit
Parts:
- removed the J5 at (195.3, 88.5)
- removed the J6 at (220.5, 88.6)
- added MCU1: DEVKIT_V1_ESP32-WROOM-32, lf_zetor_board:MODULE_DEVKIT_V1_ESP32-WROOM-32, F.Cu at (206.2, 110.0)
- J2: renamed from J9; footprint Connector_JST:JST_XH_B6B-XH-A_1x06_P2.50mm_Vertical -> Connector_JST:JST_GH_SM06B-GHS-TB_1x06-1MP_P1.25mm_Horizontal
- J3: renamed from J10; footprint Connector_JST:JST_XH_B6B-XH-A_1x06_P2.50mm_Vertical -> Connector_JST:JST_GH_SM06B-GHS-TB_1x06-1MP_P1.25mm_Horizontal
- R1, R10, R11, R12, R13, R14, R15, R16, R17, R18, R2, R3, R4, R5, R6, R7, R8, R9, U4, U9: moved to B.Cu
- SW1: value SW_DPDT -> SL19
- U10: renamed from U5; moved to B.Cu
- U11: renamed from U7; moved to B.Cu
- U3: renamed from U2; moved to B.Cu
- U5: renamed from U1; moved to B.Cu
- U6: renamed from U3; moved to B.Cu
- U7: renamed from U13; moved to B.Cu
- U8: renamed from U12; moved to B.Cu
- moved C4 185.7 mm to (241.2, 109.6)
- moved J3 179.3 mm to (228.8, 89.5), turned to 180 degrees
- moved C5 154.2 mm to (241.8, 119.8)
- moved C6 153.8 mm to (241.1, 114.8)
- moved J2 142.5 mm to (183.8, 89.5), turned to 180 degrees
- moved C3 133.2 mm to (242.3, 104.5), turned to 0 degrees
- moved R11 129.8 mm to (254.0, 44.5), turned to 90 degrees
- moved C1 128.6 mm to (179.8, 99.8), turned to 90 degrees
- moved R16 126.7 mm to (254.0, 48.5), turned to 90 degrees
- moved R10 124.6 mm to (248.8, 41.7), turned to 90 degrees
- moved R15 121.6 mm to (248.8, 45.7), turned to 90 degrees
- moved R13 110.8 mm to (235.5, 38.0), turned to 90 degrees
- moved R18 106.7 mm to (235.5, 41.8), turned to 90 degrees
- moved R9 98.2 mm to (222.5, 36.2), turned to 90 degrees
- moved R14 97.8 mm to (222.5, 40.0), turned to 90 degrees
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- renumbered C9 to C1, C7 to C2, C5 to C3, C10 to C4, C11 to C5, C12 to C6, U8 to D1, J7 to J1, J2 to J4, J4 to J5, J1 to J6, J3 to J7, U11 to U1, U10 to U2
Connections:
- J4 pad 1: LM1 -> unconnected-(J4-Pin_1-Pad1)
- J4 pad 2: LM2 -> unconnected-(J4-Pin_2-Pad2)
- J4 pad 5: unconnected-(J2-Pin_5-Pad5) -> LM2
- J4 pad 6: unconnected-(J2-Pin_6-Pad6) -> LM1
- J5 pad 1: RM1 -> unconnected-(J5-Pin_1-Pad1)
- J5 pad 2: RM2 -> unconnected-(J5-Pin_2-Pad2)
- J5 pad 5: unconnected-(J4-Pin_5-Pad5) -> RM2
- J5 pad 6: unconnected-(J4-Pin_6-Pad6) -> RM1
- J7 pad 1: VCC -> GND
- J7 pad 2: Sen9Out -> Sen6Out
- J7 pad 3: Sen8Out -> Sen7Out
- J7 pad 4: Sen7Out -> Sen8Out
- J7 pad 5: Sen6Out -> Sen9Out
- J7 pad 6: GND -> VCC
Routing:
- net S_D1: track 0.00 -> 28.6 mm
- net S_D2: track 0.00 -> 25.5 mm
- net S_D3: track 0.00 -> 22.5 mm
- net +12V: track 0.00 -> 21.6 mm
- net S_D9: track 0.00 -> 21.0 mm
- net S_D4: track 0.00 -> 19.8 mm
- net S_D8: track 0.00 -> 18.0 mm
- net S_D5: track 0.00 -> 16.3 mm
- net S_D7: track 0.00 -> 10.7 mm
- net S_D6: track 0.00 -> 9.87 mm
- added copper zone on B.Cu, net GND
Other:
- board size 128.7 x 121.5 mm -> 120 x 116.3 mm
