File: PCB/MK I/TB315A56612FNG_TO_THT/untitled.kicad_sch (KiCad schematic)
At the start: 17 parts, among them J10 Conn_01x06_Pin, J2 Conn_01x06_Pin, J4 Conn_01x06_Pin, J5 Conn_01x19_Pin, J6 Conn_01x19_Pin, J7 Conn_01x02_Pin, J9 Conn_01x06_Pin, U5 TSOP382xx, U6 DEVKIT_V1_ESP32-WROOM-32, U7 LM1086, U8 TB6612FNG

Commit message: ehhh
eeeeh
Connections:
- net GND: now also U6.15 (IO13)
Changed lines of the file:
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@@
 	(text "motor output/input with encoder encouder\n"
 		(exclude_from_sim no)
-		(at 107.315 144.145 0)
+		(at 104.775 132.715 0)
 		(effects
 			(font
@@
 	)
 	(junction
+		(at 26.67 137.16)
+		(diameter 0)
+		(color 0 0 0 0)
+	)
+	(junction
 		(at 172.72 24.13)
 		(diameter 0)
@@
 	(wire
 		(pts
+			(xy 26.67 137.16) (xy 29.21 137.16)
+		)
+		(stroke
+			(width 0)
+			(type default)
+		)
+	)
+	(wire
+		(pts
 			(xy 29.21 22.86) (xy 27.94 22.86)
 		)
@@
 	(wire
 		(pts
-			(xy 19.05 137.16) (xy 29.21 137.16)
+			(xy 19.05 137.16) (xy 26.67 137.16)
 		)
 		(stroke
@@
 	(symbol
 		(lib_id "lf_zetor_kicad_sch:DEVKIT_V1_ESP32-WROOM-32")
-		(at 127 173.99 0)
+		(at 46.99 124.46 0)
 		(unit 1)
 		(exclude_from_sim no)
@@
 		(fields_autoplaced yes)
 		(property "Reference" "U6"
-			(at 127 143.51 0)
+			(at 46.99 93.98 0)
 			(effects
 				(font
@@
 		)
 		(property "Value" "DEVKIT_V1_ESP32-WROOM-32"
-			(at 127 146.05 0)
+			(at 46.99 96.52 0)
 			(effects
 				(font
@@
 		)
 		(property "Footprint" "lf_zetor_board:MODULE_DEVKIT_V1_ESP32-WROOM-32"
-			(at 127 173.99 0)
+			(at 46.99 124.46 0)
 			(effects
 				(font
@@
 		)
 		(property "Datasheet" ""
-			(at 127 173.99 0)
+			(at 46.99 124.46 0)
 			(effects
 				(font
@@
 		)
 		(property "Description" ""
-			(at 127 173.99 0)
+			(at 46.99 124.46 0)
 			(effects
 				(font
@@
 		)
 		(property "MF" "Espressif Systems"
-			(at 127 173.99 0)
+			(at 46.99 124.46 0)
 			(effects
 				(font
@@
 		)
 		(property "Description_1" "WROOM-32 Development Board ESP32 ESP-32S WiFi Bluetooth Dev Module"
-			(at 127 173.99 0)
+			(at 46.99 124.46 0)
 			(effects
 				(font
@@
 		)
 		(property "Package" "Package"
-			(at 127 173.99 0)
+			(at 46.99 124.46 0)
 			(effects
 				(font
@@
 		)
 		(property "Price" "None"
-			(at 127 173.99 0)
+			(at 46.99 124.46 0)
 			(effects
 				(font
@@
 		)
 		(property "Check_prices" "https://www.snapeda.com/parts/DEVKIT%20V1%20ESP32-WROOM-32/Espressif+Systems/view-part/?ref=eda"
-			(at 127 173.99 0)
+			(at 46.99 124.46 0)
 			(effects
 				(font
@@
 		)
 		(property "STANDARD" "Manufacturer Recommendations"
-			(at 127 173.99 0)
+			(at 46.99 124.46 0)
 			(effects
 				(font
@@
 		)
 		(property "PARTREV" "N/A"
-			(at 127 173.99 0)
+			(at 46.99 124.46 0)
 			(effects
 				(font
@@
 		)
 		(property "SnapEDA_Link" "https://www.snapeda.com/parts/DEVKIT%20V1%20ESP32-WROOM-32/Espressif+Systems/view-part/?ref=snap"
-			(at 127 173.99 0)
+			(at 46.99 124.46 0)
 			(effects
 				(font
@@
 		)
 		(property "MP" "DEVKIT V1 ESP32-WROOM-32"
-			(at 127 173.99 0)
+			(at 46.99 124.46 0)
 			(effects
 				(font
@@
 		)
 		(property "Availability" "Not in stock"
-			(at 127 173.99 0)
+			(at 46.99 124.46 0)
 			(effects
 				(font
@@
 		)
 		(property "MANUFACTURER" "Espressif Systems"
-			(at 127 173.99 0)
+			(at 46.99 124.46 0)
 			(effects
 				(font

Commit message: saveee
s
Parts:
- C10, C12, C7, C9: footprint (none) -> Capacitor_SMD:CP_Elec_4x5.4
- J2: footprint (none) -> Connector_JST:JST_XH_B6B-XH-A_1x06_P2.50mm_Vertical
- J4: footprint Connector_JST:JST_SH_BM06B-SRSS-TB_1x06-1MP_P1.00mm_Vertical -> Connector_JST:JST_XH_B6B-XH-A_1x06_P2.50mm_Vertical
- J5, J6: footprint (none) -> Connector_PinHeader_2.54mm:PinHeader_1x19_P2.54mm_Vertical
- J7: footprint (none) -> Connector_AMASS:AMASS_XT30PW-M_1x02_P2.50mm_Horizontal
Connections:
- net +5V: now also J10.1 (Pin_1)
- net D.M.C.A.1: now also U8.21 (AIN1)
- net D.M.C.A.2: now also U8.22 (AIN2)
- net D.M.C.B.1: now also U8.17 (BIN1)
- net D.M.C.B.2: now also U8.16 (BIN2)
- net GND: now also J10.6 (Pin_6), J6.13 (Pin_13), J6.19 (Pin_19), J9.6 (Pin_6); no longer U6.15 (IO13)
- net PWM_A: now also U8.23 (PWMA)
- net PWM_B: now also U8.15 (PWMB)
- net S_D1: now also J9.5 (Pin_5)
- net S_D2: now also J9.4 (Pin_4)
- net S_D3: now also J9.3 (Pin_3)
- net S_D4: now also J9.2 (Pin_2)
- net S_D5: now also J9.1 (Pin_1)
- net S_D6: now also J10.5 (Pin_5)
- net S_D7: now also J10.4 (Pin_4)
- net S_D8: now also J10.3 (Pin_3)
- net S_D9: now also J10.2 (Pin_2)
- net LM1: now reaches U8.1 (AO1), U8.2 (AO1)
- net LM1: now also J2.1 (Pin_1)
- net RM1: now reaches U8.11 (BO1), U8.12 (BO1)
- net RM1: now also J4.5 (Pin_5)
- net LM2: now reaches U8.5 (AO2), U8.6 (AO2)
- net LM2: now also J2.2 (Pin_2)
- net RM2: now reaches U8.7 (BO2), U8.8 (BO2)
- net RM2: now also J4.6 (Pin_6)
- no-connect marks 0 -> 28
Other:
- moved on the sheet: J2, J4

Commit message: Patch some shits
Potřeby jemně předělat senzor
Parts:
- removed U6: DEVKIT_V1_ESP32-WROOM-32, lf_zetor_board:MODULE_DEVKIT_V1_ESP32-WROOM-32, symbol lf_zetor_kicad_sch:DEVKIT_V1_ESP32-WROOM-32
- added SW1: SL19, lf_zetor_board:255SB, symbol Switch:SW_DPDT_x2
- C11, C5: footprint (none) -> Capacitor_Tantalum_SMD:CP_EIA-7343-31_Kemet-D
- J2, J4: footprint Connector_JST:JST_XH_B6B-XH-A_1x06_P2.50mm_Vertical -> Connector_JST:JST_GH_SM06B-GHS-TB_1x06-1MP_P1.25mm_Horizontal
- renumbered U7 to U10, U5 to U11
Connections:
- net +12V: now also SW1.2 (B), SW1.3 (C)
- net GND: now also U8.3 (PGND1), U8.4 (PGND1)
- net RM1: now also J4.1 (Pin_1); no longer J4.5 (Pin_5)
- net RM2: now also J4.2 (Pin_2); no longer J4.6 (Pin_6)
- no-connect marks 28 -> 27

Commit message: pcb shit
Parts:
- removed J5, J6: Conn_01x19_Pin, Connector_PinHeader_2.54mm:PinHeader_1x19_P2.54mm_Vertical, symbol Connector:Conn_01x19_Pin
- added MCU1: DEVKIT_V1_ESP32-WROOM-32, lf_zetor_board:MODULE_DEVKIT_V1_ESP32-WROOM-32, symbol lf_zetor_kicad_sch:DEVKIT_V1_ESP32-WROOM-32
- J2: renamed from J9; footprint Connector_JST:JST_XH_B6B-XH-A_1x06_P2.50mm_Vertical -> Connector_JST:JST_GH_SM06B-GHS-TB_1x06-1MP_P1.25mm_Horizontal
- J3: renamed from J10; footprint Connector_JST:JST_XH_B6B-XH-A_1x06_P2.50mm_Vertical -> Connector_JST:JST_GH_SM06B-GHS-TB_1x06-1MP_P1.25mm_Horizontal
- renumbered C9 to C1, C7 to C2, C5 to C3, C10 to C4, C11 to C5, C12 to C6, U8 to D1, J7 to J1, J2 to J4, J4 to J5, U11 to U1, U10 to U2
Connections:
- net +5V: now also MCU1.19 (EXT_5V)
- net D-pin-ESP: now also MCU1.3 (SENSOR_VP)
- net D.M.C.A.1: now also MCU1.23 (IO15)
- net D.M.C.A.2: now also MCU1.24 (IO2)
- net D.M.C.B.1: now also MCU1.25 (IO0)
- net D.M.C.B.2: now also MCU1.26 (IO4)
- net GND: now also MCU1.14 (GND1), MCU1.32 (GND2), MCU1.38 (GND3)
- net LM1: now also J4.6 (Pin_6); no longer J4.1 (Pin_1)
- net LM2: now also J4.5 (Pin_5); no longer J4.2 (Pin_2)
- net PWM_A: now also MCU1.13 (IO12)
- net PWM_B: now also MCU1.15 (IO13)
- net RM1: now also J5.6 (Pin_6); no longer J5.1 (Pin_1)
- net RM2: now also J5.5 (Pin_5); no longer J5.2 (Pin_2)
- net S_D1: now also MCU1.12 (IO14)
- net S_D2: now also MCU1.11 (IO27)
- net S_D3: now also MCU1.10 (IO26)
- net S_D4: now also MCU1.9 (IO25)
- net S_D5: now also MCU1.8 (IO33)
- net S_D6: now also MCU1.37 (IO23)
- net S_D7: now also MCU1.36 (IO22)
- net S_D8: now also MCU1.31 (IO19)
- net S_D9: now also MCU1.30 (IO18)
- no-connect marks 27 -> 23
