File: PCB/MK I/senzor_ring/senzor_ring.kicad_sch (KiCad schematic)
At the start: 29 parts, among them J1 Conn_01x06_Pin, J2 Conn_01x06_Pin, U1 QRE1113GR, U2 QRE1113GR, U3 QRE1113GR, U4 QRE1113GR, U5 QRE1113GR, U6 QRE1113GR, U7 QRE1113GR, U8 QRE1113GR, U9 QRE1113GR

Commit message: Patch some shits
Potřeby jemně předělat senzor
Parts:
- renumbered J2 to J3, R3 to R1, R15 to R10, R17 to R11, R9 to R12, R12 to R14, R16 to R15, R18 to R16, R10 to R17, R14 to R18, R7 to R2, R1 to R3, R5 to R4, R4 to R5, R8 to R6, R2 to R7, R6 to R8, R11 to R9, U8 to U12, U6 to U13
Connections:
- net GND: now also J1.6 (Pin_6), J3.6 (Pin_6)
- net Sen1Out: now also J1.5 (Pin_5)
- net Sen2Out: now also J1.4 (Pin_4)
- net Sen3Out: now also J1.3 (Pin_3)
- net Sen4Out: now also J1.2 (Pin_2)
- net Sen5Out: now also J1.1 (Pin_1)
- net Sen6Out: now also J3.5 (Pin_5)
- net Sen7Out: now also J3.4 (Pin_4)
- net Sen8Out: now also J3.3 (Pin_3)
- net Sen9Out: now also J3.2 (Pin_2)
- net VCC: now also J3.1 (Pin_1)
Other:
- note added: "Senzor Outpout Conectors"
- note removed: "motor output/input with encoder encouder"
- moved on the sheet: J1, J3

Commit message: pcb shit
Parts:
- renumbered J1 to J6, J3 to J7, U5 to U10, U7 to U11, U2 to U3, U1 to U5, U3 to U6, U13 to U7, U12 to U8
Connections:
- net GND: now also J7.1 (Pin_1); no longer J7.6 (Pin_6)
- net Sen6Out: now also J7.2 (Pin_2); no longer J7.5 (Pin_5)
- net Sen7Out: now also J7.3 (Pin_3); no longer J7.4 (Pin_4)
- net Sen8Out: now also J7.4 (Pin_4); no longer J7.3 (Pin_3)
- net Sen9Out: now also J7.5 (Pin_5); no longer J7.2 (Pin_2)
- net VCC: now also J7.6 (Pin_6); no longer J7.1 (Pin_1)
Other:
- note added: "VCC = +5v"
