File: PCB/MK I/FL-Zetor/FL-Zetor-Senzor/FL-Zetor-Senzor.kicad_pcb (KiCad board)
At the start: 2 copper layers, 115 x 21.2 mm, 32 parts, among them J1 Conn_01x06_Pin, J2 Conn_01x06_Pin, U1 QRE1113GR, U2 QRE1113GR, U3 QRE1113GR, U4 QRE1113GR, U5 QRE1113GR, U6 QRE1113GR, U7 QRE1113GR, U8 QRE1113GR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

Commit message: update for senzot + grb files
Routing:
- net GND: track 0.00 -> 64.2 mm, vias 0 -> 5
- net Sen4Out: track 17.9 -> 20.0 mm
- net Sen5Out: track 31.2 -> 30.3 mm
- net Sen1Out: track 38.7 -> 37.9 mm
