File: PCB/MK I/FL-Zetor/FL-Zetor.kicad_pcb (KiCad board)
At the start: 2 copper layers, 120 x 116.3 mm, 45 parts, among them J1 Conn_01x02_Pin, J2 Conn_01x06_Pin, J3 Conn_01x06_Pin, J4 Conn_01x06_Pin, J5 Conn_01x06_Pin, J6 Conn_01x06_Pin, J7 Conn_01x06_Pin, SW1 SL19, U1 TSOP382xx, U10 QRE1113GR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

Commit message: pcbs done
that pieces of craps is done
Parts:
- removed J6, J7: Conn_01x06_Pin, Connector_JST:JST_GH_SM06B-GHS-TB_1x06-1MP_P1.25mm_Horizontal
- removed R1, R10, R11, R12, R13, R2, R3, R4, R9: 100R, Resistor_SMD:R_0805_2012Metric
- removed R14, R15, R16, R17, R18, R5, R6, R7, R8: 10k, Resistor_SMD:R_0805_2012Metric
- removed U10, U11, U3, U4, U5, U6, U7, U8, U9: QRE1113GR, OptoDevice:OnSemi_CASE100CY
- added G***: LOGO, lf_zetor_graphic:SHIKANOKO_IMG, F.Cu at (173.0, 122.5)
- added G***: LOGO, lf_zetor_graphic:SPS_LOGO_IMG, F.Cu at (107.2, 123.0)
- added H1: MountingHole_Pad, MountingHole:MountingHole_3.2mm_M3_ISO7380_Pad, F.Cu at (94.4, 123.8)
- added H2: MountingHole_Pad, MountingHole:MountingHole_3.2mm_M3_ISO7380_Pad, F.Cu at (94.4, 100.8)
- added H3: MountingHole_Pad, MountingHole:MountingHole_3.2mm_M3_ISO7380_Pad, F.Cu at (183.9, 72.0)
- added H4: MountingHole_Pad, MountingHole:MountingHole_3.2mm_M3_ISO7380_Pad, F.Cu at (114.9, 72.0)
- added H5: MountingHole_Pad, MountingHole:MountingHole_3.2mm_M3_ISO7380_Pad, F.Cu at (204.4, 100.8)
- added H6: MountingHole_Pad, MountingHole:MountingHole_3.2mm_M3_ISO7380_Pad, F.Cu at (204.4, 123.8)
- C3, C5: footprint Capacitor_Tantalum_SMD:CP_EIA-7343-31_Kemet-D -> Capacitor_SMD:C_0805_2012Metric_Pad1.18x1.45mm_HandSolder
- J1: footprint Connector_AMASS:AMASS_XT30PW-M_1x02_P2.50mm_Horizontal -> Connector_AMASS:AMASS_XT30U-F_1x02_P5.0mm_Vertical
- moved C5 89.6 mm to (152.5, 112.5)
- moved C3 89.5 mm to (153.0, 100.2)
- moved C4 87.4 mm to (154.0, 103.8)
- moved C6 87.4 mm to (153.9, 109.0)
- moved D1 87.3 mm to (144.9, 106.5)
- moved SW1 70.4 mm to (114.1, 98.3), turned to 90 degrees
- moved C2 69.3 mm to (117.9, 81.5)
- moved C1 69.3 mm to (112.9, 81.6)
- moved U2 69.3 mm to (119.2, 86.9)
- moved J1 61.0 mm to (121.4, 103.8), turned to 0 degrees
- moved J2 59.5 mm to (126.9, 72.0)
- moved J3 59.5 mm to (171.9, 72.0)
- moved J4 59.5 mm to (113.9, 112.3)
- moved J5 59.5 mm to (184.9, 112.5)
- moved MCU1 59.5 mm to (149.4, 92.5)
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Connections:
- MCU1 pad 23: D.M.C.A.1 -> D.M.C.B.2
- MCU1 pad 24: D.M.C.A.2 -> D.M.C.B.1
- MCU1 pad 25: D.M.C.B.1 -> D.M.C.A.1
- MCU1 pad 26: D.M.C.B.2 -> D.M.C.A.2
Routing:
- net +5V: track 0.00 -> 130.5 mm
- net D-pin-ESP: track 0.00 -> 62.1 mm, vias 0 -> 2
- net +12V: track 21.6 -> 77.3 mm
- net RM2: track 0.00 -> 46.3 mm, vias 0 -> 2
- net RM1: track 0.00 -> 44.2 mm, vias 0 -> 2
- net LM2: track 0.00 -> 33.2 mm, vias 0 -> 2
- net LM1: track 0.00 -> 31.2 mm, vias 0 -> 2
- net GND: track 0.00 -> 21.5 mm
- net D.M.C.A.2: track 0.00 -> 19.7 mm, vias 0 -> 1
- net D.M.C.A.1: track 0.00 -> 19.2 mm, vias 0 -> 1
- net D.M.C.B.1: track 0.00 -> 18.5 mm, vias 0 -> 1
- net D.M.C.B.2: track 0.00 -> 17.4 mm, vias 0 -> 1
- net PWM_B: track 0.00 -> 13.3 mm, vias 0 -> 1
- net PWM_A: track 0.00 -> 13.2 mm, vias 0 -> 1
- added copper zone on F.Cu, net +5V
- added copper zone on F.Cu, net GND
Other:
- board size 120 x 116.3 mm -> 120 x 65 mm
- board text added: "LF-Zetor MKI"
- board text added: "Made by Bobutek team"

Commit message: update for senzot + grb files
Other:
- board text added: "L-Motor"
- board text added: "R-Motor"
Changed lines of the file:
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@@
 			(drillshape 0)
 			(scaleselection 1)
-			(outputdirectory "../../../../../Downloads/")
+			(outputdirectory "../GRB-Files/Main/")
 		)
 	)
@@
 	)
 	(gr_line
+		(start 109.375 119.025)
+		(end 109.375 105.525)
+		(stroke
+			(width 0.2)
+			(type default)
+		)
+		(layer "F.Cu")
+	)
+	(gr_line
+		(start 89.375 119.025)
+		(end 109.375 119.025)
+		(stroke
+			(width 0.2)
+			(type default)
+		)
+		(layer "F.Cu")
+	)
+	(gr_line
+		(start 109.375 105.525)
+		(end 89.35 105.525)
+		(stroke
+			(width 0.2)
+			(type default)
+		)
+		(layer "F.Cu")
+	)
+	(gr_line
+		(start 189.375 119.025)
+		(end 209.35 119.025)
+		(stroke
+			(width 0.2)
+			(type solid)
+		)
+		(layer "F.SilkS")
+	)
+	(gr_line
+		(start 189.375 105.5)
+		(end 189.375 119.025)
+		(stroke
+			(width 0.2)
+			(type solid)
+		)
+		(layer "F.SilkS")
+	)
+	(gr_line
+		(start 209.375 105.525)
+		(end 189.375 105.5)
+		(stroke
+			(width 0.2)
+			(type solid)
+		)
+		(layer "F.SilkS")
+	)
+	(gr_line
 		(start 109.37 119.025)
 		(end 109.37 105.525)
@@
 	(gr_arc
 		(start 113.40555 68.48945)
-		(mid 115.027649 67.405592)
+		(mid 115.02766 67.405599)
 		(end 116.941068 67.025)
 		(stroke
@@
 	(gr_arc
 		(start 181.7989 67.025)
-		(mid 183.712342 67.405613)
+		(mid 183.721145 67.409277)
 		(end 185.347967 68.502967)
 		(stroke
@@
 	(gr_arc
 		(start 89.37 94.59613)
-		(mid 89.750613 92.682658)
+		(mid 89.750601 92.682646)
 		(end 90.83451 91.06049)
 		(stroke
@@
 	(gr_arc
 		(start 207.90555 91.06055)
-		(mid 208.989408 92.682649)
+		(mid 208.989401 92.68266)
 		(end 209.37 94.596068)
 		(stroke
@@
 		)
 	)
+	(gr_text "L-Motor"
+		(at 108.75 118.9 90)
+		(layer "F.SilkS" knockout)
+		(effects
+			(font
+				(size 2 2)
+				(thickness 0.4)
+				(bold yes)
+			)
+			(justify left bottom)
+		)
+	)
+	(gr_text "R-Motor"
+		(at 190 105.5 270)
+		(layer "F.SilkS" knockout)
+		(effects
+			(font
+				(size 2 2)
+				(thickness 0.4)
+				(bold yes)
+			)
+			(justify left bottom)
+		)
+	)
 	(gr_text "Made by Bobutek team"
 		(at 198.25 128.75 0)
@@
 	)
 	(group "Main"
-		(members "06417e62-ec4b-4d41-a049-e50fadd3d77f" "25e05c6c-248d-445e-91c1-e789fdea496c"
-			"41f8330f-cab4-4b45-9974-347731629796" "43582b94-3e0d-4086-9525-bb1b606aeaf9"
-			"46ca1b62-1b69-40d0-a60b-fe06007473d6" "4f7416b4-be13-4370-934d-4e55188dbc60"
-			"52fcd11d-e7d2-4dc9-9584-93ca63da640d" "59a52631-0c21-4fb9-9f7d-a4d97479cdd1"
-			"5f9c7168-504c-4ba6-8fc9-d4d2f968a717" "6e25dc86-008a-4fd2-9a16-d08ef54fbd47"
-			"756f6ea9-570f-4a94-9e48-2ec84cd0dc10" "75d408fd-887c-430d-b84f-76a93db9cfa8"
-			"8158888d-a2f9-46d0-951e-4c51eef44335" "86736a73-4613-4638-a9e6-984dd20f848e"
-			"8e163e1b-baf7-4683-957b-8483aab60783" "9106288a-1b7e-4123-89bc-4869280db91d"
+		(members "0428aea6-aeef-4983-97d1-9b24e09e9c3b" "06417e62-ec4b-4d41-a049-e50fadd3d77f"
+			"1e77404a-04b6-4002-afd9-89c174a966d2" "25e05c6c-248d-445e-91c1-e789fdea496c"
+			"2dead5da-5ca7-499d-ab23-eb61bfa08e78" "41f8330f-cab4-4b45-9974-347731629796"
+			"43582b94-3e0d-4086-9525-bb1b606aeaf9" "46ca1b62-1b69-40d0-a60b-fe06007473d6"
+			"4f7416b4-be13-4370-934d-4e55188dbc60" "52fcd11d-e7d2-4dc9-9584-93ca63da640d"
+			"59a52631-0c21-4fb9-9f7d-a4d97479cdd1" "5f9c7168-504c-4ba6-8fc9-d4d2f968a717"
+			"6e25dc86-008a-4fd2-9a16-d08ef54fbd47" "756f6ea9-570f-4a94-9e48-2ec84cd0dc10"
+			"75d408fd-887c-430d-b84f-76a93db9cfa8" "8158888d-a2f9-46d0-951e-4c51eef44335"
+			"86736a73-4613-4638-a9e6-984dd20f848e" "8e163e1b-baf7-4683-957b-8483aab60783"
+			"9106288a-1b7e-4123-89bc-4869280db91d" "a1416e4f-e4fb-462f-b069-9ddb39375cc5"
 			"c53f2388-314f-45cb-a51c-7798e422d79b" "c5593b0c-26d6-44e9-bbe8-d722bd6bd7f1"
-			"c7084561-50b1-45d1-99d2-1daca36f127c" "e3d5f1ee-af64-46bb-8b30-902027877ccc"
-			"e6264155-f2b4-4f4d-9190-8a7603b42d19" "f09b90f0-36c6-43a3-a7da-149896e91428"
-			"f6abfb8a-c4d8-4c70-898e-86b3df9424f0" "f9102673-7e7f-4aa1-a62c-c8a1bb4de9d2"
+			"c7084561-50b1-45d1-99d2-1daca36f127c" "cc729f12-0fa3-4bf4-be7e-6a2021e62310"
+			"e3d5f1ee-af64-46bb-8b30-902027877ccc" "e6264155-f2b4-4f4d-9190-8a7603b42d19"
+			"f09b90f0-36c6-43a3-a7da-149896e91428" "f6abfb8a-c4d8-4c70-898e-86b3df9424f0"
+			"f8edcddc-bbfb-4a76-a6cd-42b727eaa0f4" "f9102673-7e7f-4aa1-a62c-c8a1bb4de9d2"
 		)
 	)

Commit message: some shit
Parts:
- added G***: LOGO, LOGO, F.Cu at (184.6, 93.9)
